File: tinyLIPO.brd (EAGLE design)
At the start: 30 x 18 mm, 13 parts, among them IC1 MCP73831

Commit message: removed gerber schematic place adjustments added r4 r4,r3 from 220e to 470e board T.NAME adjust no DRC no ERC
Signed-off-by: kaushalpkk <kaushal.panduru@gmail.com>
Parts:
- added R4: 470e, rcl:M0805
- BATT1: value (none) -> JST 2mm
- BATT2: value (none) -> JST2.54mm
- C1, C2: value (none) -> 4.7uF
- CHG: value (none) -> red
- POW: value (none) -> green
- R1: value (none) -> 2.2k
- R2: value (none) -> 10k
- R3: value (none) -> 470e
- SW1: value (none) -> switch
- USB: value (none) -> micro USB
Connections:
- new net N$7: POW.C, R4.2
- net GND: now also R4.1; no longer POW.C
Routing:
- net N$7: track 0.00 -> 2.00 mm
